File: EggtimerIon.kicad_sch (KiCad schematic)
At the start: 46 parts, among them J1 Conn_01x02, J2 Conn_01x03, J3 B2B-PH-K-S, J4 USB_C_Receptacle_USB2.0, Q1 IRLML6244, Q2 2N7002, Q3 2N7002, U1 ESP32-WROOM-32-N4, U2 MPU-6050, U3 MS5611-01BA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

Commit message: Completed first round of layout
Did a lot of stuff here ok?
Parts:
- U1: footprint ESP32-WROOM-32-N4:MOD_ESP32-WROOM-32_EXP -> RF_Module:ESP32-WROOM-32
Connections:
- net IO12: now also Q1.1 (G)
- net IO18: no longer Q1.1 (G)
- net USB_D-: now reaches D1.3 (K), J4.A7 (D-), J4.B7 (D-), U6.5 (D-)
- net USB_D+: now reaches D1.4 (K), J4.A6 (D+), J4.B6 (D+), U6.4 (D+)
Changed lines of the file:
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@@
 	)
 	(no_connect
-		(at 63.5 154.94)
+		(at 135.89 165.1)
 	)
 	(no_connect
@@
 		)
 	)
+	(label "USB_D+"
+		(at 46.99 60.96 0)
+		(effects
+			(font
+				(size 1.27 1.27)
+			)
+			(justify left bottom)
+		)
+	)
 	(label "SD2"
 		(at 63.5 162.56 0)
@@
 		)
 	)
+	(label "USB_D-"
+		(at 46.99 55.88 0)
+		(effects
+			(font
+				(size 1.27 1.27)
+			)
+			(justify left bottom)
+		)
+	)
 	(label "SDA"
 		(at 201.93 125.73 0)
@@
 		)
 	)
-	(label "IO18"
+	(label "IO12"
 		(at 195.58 66.04 180)
 		(effects
@@
 			)
 		)
-		(property "Footprint" "ESP32-WROOM-32-N4:MOD_ESP32-WROOM-32_EXP"
+		(property "Footprint" "RF_Module:ESP32-WROOM-32"
 			(at 76.2 121.92 0)
 			(effects
