File: EggtimerIon.kicad_pcb (KiCad board)
At the start: 4 copper layers, 45 x 30 mm, 29 parts, among them J1 Conn_01x02, J2 Conn_01x03, J3 B2B-PH-K-S, Q1 IRLML6244, U1 ESP32-WROOM-32-N4, U2 MPU-6050, U3 MS5611-01BA, U5 AP2112K-3.3

Commit message: work
Parts:
- removed U1: ESP32-WROOM-32-N4, RF_Module:ESP32-WROOM-32
- added J4: USB_C_Receptacle_USB2.0_16P, Connector_USB:USB_C_Receptacle_Palconn_UTC16-G, F.Cu at (151.1, 121.0)
- added U4: ESP32-S3-WROOM-1-N16, Morten_Library:ESP32-S3-WROOM-1, F.Cu at (142.4, 95.3)
Routing:
- net /SDA: track 51.7 -> 0.00 mm, vias 4 -> 0
- net /SCL: track 48.7 -> 0.00 mm, vias 3 -> 0
- net /RXD0: track 46.9 -> 0.00 mm, vias 2 -> 0
- net /TXD0: track 46.1 -> 0.00 mm, vias 2 -> 0
- net GND: track 30.4 -> 0.00 mm, vias 17 -> 0
- net /IO0: track 25.8 -> 0.00 mm, vias 1 -> 0
- net Net-(Q1-D): track 10.3 -> 0.00 mm
- net /IO12: track 9.32 -> 0.00 mm
- net BAT+: track 9.00 -> 0.00 mm
- net Net-(LS1-Pad1): track 4.81 -> 0.00 mm
- net /EN: track 4.45 -> 0.00 mm
- net Net-(U5-VIN): track 3.51 -> 0.00 mm
- net +3V3: track 2.33 -> 0.00 mm
- net Net-(U2-REGOUT): track 1.91 -> 0.00 mm
- net Net-(U2-CPOUT): track 1.90 -> 0.00 mm

Commit message: Routing Updates to parts
Parts:
- removed J1: Conn_01x02, Connector_PinHeader_2.54mm:PinHeader_1x02_P2.54mm_Vertical
- removed J2: Conn_01x03, Connector_PinHeader_2.54mm:PinHeader_1x03_P2.54mm_Vertical
- removed R10: 10k, Capacitor_SMD:C_0402_1005Metric
- added D1: LED, LED_SMD:LED_0603_1608Metric, F.Cu at (171.0, 113.9)
- added D2: LED, LED_SMD:LED_0603_1608Metric, F.Cu at (171.0, 111.9)
- added R12: 5.1k, Resistor_SMD:R_0402_1005Metric, F.Cu at (158.6, 110.0)
- added R16: 27, Resistor_SMD:R_0402_1005Metric, F.Cu at (153.5, 106.2)
- added R17: 27, Resistor_SMD:R_0402_1005Metric, F.Cu at (152.5, 106.2)
- added R5: 10k, Capacitor_SMD:C_0402_1005Metric, F.Cu at (157.4, 102.3)
- added R6: 5.1k, Resistor_SMD:R_0402_1005Metric, F.Cu at (158.6, 112.0)
- added R7: 1.5k, Capacitor_SMD:C_0402_1005Metric, F.Cu at (167.9, 112.2)
- added SW1: RESET, Button_Switch_SMD:SW_SPST_B3U-1000P, F.Cu at (144.9, 109.1)
- added SW2: BOOT, Button_Switch_SMD:SW_SPST_B3U-1000P, F.Cu at (162.5, 112.4)
- C3: value TBD -> 1uF
- C8: value 100nF -> 0.1uF
- CR1: footprint MBRS130L3TG:DIODE_SMB_2L_ONS -> Diode:DIODE_SMB_2L_ONS
- R1: value TBD -> 2k
- R2, R3: value TBD -> 4.7k
- R4: value R -> 1k
- U4: value ESP32-S3-WROOM-1-N16 -> ESP32-S3-WROOM-1-N8; footprint Morten_Library:ESP32-S3-WROOM-1 -> RF_Module:ESP32-S3-WROOM-1
- U5: footprint Package_TO_SOT_SMD:SOT-23-5 -> LDO:SOT_RG1_DIO
- moved R1 27.9 mm to (167.9, 113.9), turned to 0 degrees
- moved C8 16.4 mm to (166.9, 105.2), turned to -90 degrees
- moved J4 10.2 mm to (152.5, 110.9)
- moved C4 9.71 mm to (169.7, 100.4), turned to -90 degrees
- moved U3 9.65 mm to (163.5, 105.9), turned to -90 degrees
- moved C7 9.47 mm to (169.7, 98.4), turned to 90 degrees
- moved Q1 8.77 mm to (170.7, 108.0)
- moved C5 7.86 mm to (167.7, 95.9), turned to 180 degrees
- moved U2 4.06 mm to (165.9, 99.0), turned to 90 degrees
- moved U5 3.57 mm to (173.9, 94.5)
- moved C11 3.54 mm to (177.0, 94.0), turned to -90 degrees
- moved R2 2.91 mm to (160.7, 100.9), turned to 90 degrees
- moved LS1 2.28 mm to (175.7, 102.4)
- moved C6 2.17 mm to (162.5, 97.1), turned to 90 degrees
- moved R4 2.05 mm to (178.8, 97.4)
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Connections:
- C3 pad 1: GND -> /ESP_EN
- C3 pad 2: /EN -> GND
- J4 pad A1: (no net) -> GND
- J4 pad A12: (no net) -> GND
- J4 pad A4: (no net) -> unconnected-(J4-VBUS-PadA4)_2
- J4 pad A5: (no net) -> Net-(J4-CC1)
- J4 pad A6: (no net) -> USB_D+
- J4 pad A7: (no net) -> USB_D-
- J4 pad A8: (no net) -> unconnected-(J4-SBU1-PadA8)
- J4 pad B1: (no net) -> GND
- J4 pad B12: (no net) -> GND
- J4 pad B4: (no net) -> unconnected-(J4-VBUS-PadA4)_3
- J4 pad B5: (no net) -> Net-(J4-CC2)
- J4 pad B6: (no net) -> USB_D+
- J4 pad B7: (no net) -> USB_D-
- J4 pad B8: (no net) -> unconnected-(J4-SBU2-PadB8)
- J4 pad S1: (no net) -> GND
- Q1 pad 1: /IO12 -> /BUZZER
- R1 pad 1: +3V3 -> /LED
- R1 pad 2: /EN -> Net-(D1-A)
- R11 pad 1: +3V3 -> /ESP_EN
- R11 pad 2: /EN -> +3V3
- U3 pad 4: unconnected-(U3-CSB-Pad4) -> GND
- U3 pad 5: unconnected-(U3-CSB-Pad4)_1 -> GND
- U4 pad 13: /USB_D- -> USB_D-
- U4 pad 14: /USB_D+ -> USB_D+
- U4 pad 18: /CS -> unconnected-(U4-GPIO10-Pad18)
- U4 pad 19: /MOSI -> unconnected-(U4-GPIO11-Pad19)
- U4 pad 20: /CLK -> unconnected-(U4-GPIO12-Pad20)
- U4 pad 21: /MISO -> unconnected-(U4-GPIO13-Pad21)
- U4 pad 22: /RESET -> unconnected-(U4-GPIO14-Pad22)
- U4 pad 25: /USER_SW -> unconnected-(U4-GPIO48-Pad25)
- U4 pad 32: /R_LED -> /LED
- U4 pad 33: /G_LED -> /BUZZER
- U4 pad 34: /B_LED -> unconnected-(U4-GPIO41-Pad34)
- U4 pad 36: /ESP_RXD -> unconnected-(U4-RXD0/U0RXD/GPIO44-Pad36)
- U4 pad 37: /ESP_TXD -> unconnected-(U4-TXD0/U0TXD/GPIO43-Pad37)
- U4 pad 8: /IRQ -> unconnected-(U4-GPIO15-Pad8)
Routing:
- net (no net): track 0.00 -> 30.4 mm, vias 0 -> 4
- net /SDA: track 0.00 -> 27.4 mm, vias 0 -> 3
- net /SCL: track 0.00 -> 24.2 mm, vias 0 -> 2
- net Net-(J4-CC1): track 0.00 -> 9.12 mm
- net GND: track 0.00 -> 6.67 mm, vias 0 -> 6
- net /ESP_IO0: track 0.00 -> 6.29 mm, vias 0 -> 2
- net Net-(J4-CC2): track 0.00 -> 6.10 mm
- net BAT+: track 0.00 -> 5.62 mm
- net /ESP_EN: track 0.00 -> 5.07 mm
- net +3V3: track 0.00 -> 4.54 mm
- net USB_D+: track 0.00 -> 3.43 mm
- net USB_D-: track 0.00 -> 3.43 mm
- net Net-(U4-GPIO3): track 0.00 -> 2.04 mm
Other:
- board text added: "BOOT"
- board text added: "RST"
- board text removed: "GND"
- board text removed: "IO"
- board text removed: "RX"
- board text removed: "TX"

Commit message: updates
Parts:
- moved SW2 0.81 mm to (163.3, 112.5)
- moved R1 0.51 mm to (168.2, 113.5)
- moved R7 0.32 mm to (168.2, 112.3)
- moved D1 0.23 mm to (170.9, 113.7), turned to 180 degrees
- moved C5 0.15 mm to (167.6, 95.8)
- moved D2 0.13 mm to (170.9, 112.0), turned to 180 degrees
- moved C1 0.10 mm to (137.8, 106.0)
- moved C2 0.10 mm to (137.8, 107.0)
- turned C3 to -90 degrees
- turned R11 to -90 degrees
Connections:
- C1 pad 1: GND -> BAT-
- C10 pad 2: GND -> BAT-
- C11 pad 2: GND -> BAT-
- C2 pad 1: GND -> BAT-
- C3 pad 2: GND -> BAT-
- C4 pad 1: GND -> BAT-
- C5 pad 1: GND -> BAT-
- C6 pad 2: GND -> BAT-
- C7 pad 2: GND -> BAT-
- C8 pad 2: GND -> BAT-
- D1 pad 1: GND -> BAT-
- D2 pad 1: GND -> BAT-
- J4 pad A1: GND -> BAT-
- J4 pad A12: GND -> BAT-
- J4 pad B1: GND -> BAT-
- J4 pad B12: GND -> BAT-
- J4 pad S1: GND -> BAT-
- Q1 pad 2: GND -> BAT-
- R12 pad 2: GND -> BAT-
- R6 pad 1: GND -> BAT-
- SW1 pad 1: GND -> BAT-
- SW2 pad 1: GND -> BAT-
- U2 pad 1: GND -> BAT-
- U2 pad 11: GND -> BAT-
- U2 pad 18: GND -> BAT-
- U2 pad 9: GND -> BAT-
- U3 pad 3: GND -> BAT-
- U3 pad 4: GND -> BAT-
- U3 pad 5: GND -> BAT-
- U4 pad 1: GND -> BAT-
- U4 pad 40: GND -> BAT-
- U4 pad 41: GND -> BAT-
- U5 pad 2: GND -> BAT-
Routing:
- net /LED: track 0.00 -> 40.7 mm, vias 0 -> 2
- net /ESP_IO0: track 6.29 -> 42.4 mm
- net /BUZZER: track 0.00 -> 33.6 mm, vias 0 -> 2
- net BAT-: track 0.00 -> 32.9 mm, vias 0 -> 22
- net (no net): track 30.4 -> 0.00 mm, vias 4 -> 0
- net GND: track 6.67 -> 0.00 mm, vias 6 -> 0
- net Net-(Q1-D): track 0.00 -> 6.25 mm
- net Net-(LS1-Pad1): track 0.00 -> 5.05 mm
- net Net-(U5-VIN): track 0.00 -> 3.44 mm
- net /ESP_EN: track 5.07 -> 7.53 mm
- net BAT+: track 5.62 -> 7.90 mm
- net Net-(U2-REGOUT): track 0.00 -> 1.91 mm
- net Net-(U2-CPOUT): track 0.00 -> 1.73 mm
- net Net-(D2-A): track 0.00 -> 1.56 mm
- net Net-(D1-A): track 0.00 -> 1.52 mm
- added copper zone on B.Cu, net BAT-
- removed copper zone on B.Cu, net GND
- removed copper zone on In1.Cu, net GND
- removed copper zone on In2.Cu, net GND
Other:
- copper layers 4 -> 2

Commit message: Update Footprints
Connections:
- U5 pad 3: unconnected-(U5-EN-Pad3) -> +3V3
Routing:
- net USB_D+: track 3.60 -> 6.08 mm
- net USB_D-: track 3.59 -> 5.38 mm

Commit message: Updates
Parts:
- H3: footprint PCM_JLCPCB:Hole, 3mm -> Mount:hole
- U4: footprint RF_Module:ESP32-S3-WROOM-1 -> ESP:ESP32-S3-WROOM-1_EXP
Routing:
- net BAT-: vias 22 -> 31
