File: F25.kicad_pcb (KiCad board)
At the start: 2 copper layers, 45 x 30 mm, 37 parts, among them J3 B2B-PH-K-S, J4 USB_C_Receptacle_USB2.0_16P, Q1 IRLML6244, SW1 RESET, SW2 BOOT, U2 MPU-6050, U3 MS5611-01BA, U4 ESP32-S3-WROOM-1-N8, U5 AP2112K-3.3

Commit message: General Updates
Parts:
- H1, H2: footprint PCM_JLCPCB:Hole, 3mm -> Mount:hole
- U4: footprint ESP:ESP32-S3-WROOM-1_EXP -> RF_Module:ESP32-S3-WROOM-1
- moved C8 0.15 mm to (166.8, 105.2)
- moved H1 0.08 mm to (176.9, 89.1)
Routing:
- net BAT-: track 32.9 -> 38.3 mm, vias 31 -> 23
- net USB_D-: track 5.38 -> 5.97 mm
