File: kicad/F25.kicad_pcb (KiCad board)
At the start: 2 copper layers, 45 x 30 mm, 37 parts, among them J3 B2B-PH-K-S, J4 USB_C_Receptacle_USB2.0_16P, Q1 IRLML6244, SW1 RESET, SW2 BOOT, U1 MS5611-01BA, U2 MPU-6050, U4 ESP32-S3-WROOM-1-N8, U5 AP2112K-3.3

Commit message: Update Silk to SVG
Other:
- board text removed: "BOOT"
- board text removed: "MAV"
- board text removed: "RST"
