File: kicad/F25.kicad_sch (KiCad schematic)
At the start: 37 parts, among them J3 B2B-PH-K-S, J4 USB_C_Receptacle_USB2.0_16P, Q1 IRLML6244, SW1 RESET, SW2 BOOT, U1 MS5611-01BA, U2 MPU-6050, U4 ESP32-S3-WROOM-1-N8, U5 AP2112K-3.3

Commit message: MAJOR UPDATES
Parts:
- removed C11: 1uF, Capacitor_SMD:C_0402_1005Metric, symbol Device:C
- added C8: 10uF, Capacitor_SMD:C_0402_1005Metric, symbol Device:C
- added Q2: DMG3415U, Package_TO_SOT_SMD:SOT-23, symbol Transistor_FET:DMG2301L
- added R8, R9: 100k, Capacitor_SMD:C_0402_1005Metric, symbol Device:R
- C10: value 1uF -> 10uF; LCSC C52923 -> C15525
- H1, H2, H3: symbol Mechanical:MountingHole -> Mechanical:MountingHole_Pad
- R5: value 10k -> 100k; LCSC C25744 -> C25741
Connections:
- net +3V3: now also C10.2; no longer R5.2, U5.3 (EN)
- net BAT+: now also Q2.3 (D); no longer C10.1, CR1.2
- net BUZZER: now also R8.1
- net GND: now also C10.1, H1.1, H2.1, H3.1, C8.1, R8.2, R9.1; no longer C10.2
- net VBUS: now reaches J4.A4 (VBUS), J4.A9 (VBUS), J4.B4 (VBUS), J4.B9 (VBUS)
- net VBUS: now also CR1.2, Q2.1 (G), R9.2
- net at CR1.1, U5.1 (VIN): now also R5.1, C8.2, Q2.2 (S)
- net at U4.15 (GPIO3): no longer R5.1
- new net: R5.2, U5.3 (EN)
Other:
- moved on the sheet: CR1, D2, R7, U5

Commit message: MAJOR FIXES
Fixed Power circuitry
Added usb power support
Added pulldown to buzzer (thx taz)
Removed 10k pullup on gpio3
Parts:
- Q2: LCSC (none) -> C7202986
Changed lines of the file:
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@@
+			)
+		)
+		(property "LCSC" "C7202986"
+			(at 58.42 166.37 0)
+			(effects
+				(font
+					(size 1.27 1.27)
+				)
+				(hide yes)
 			)
 		)
